File: stm32g474/stm32g474.kicad_pcb (KiCad board)
At the start: 4 copper layers, 0 parts

Commit message: pcb update
Parts:
- added C1: 100n, Capacitor_SMD:C_0402_1005Metric, F.Cu at (150.5, 90.5)
- added C10: 10u, Capacitor_SMD:C_0805_2012Metric, F.Cu at (131.2, 97.8)
- added C11: 10n, Capacitor_SMD:C_0402_1005Metric, F.Cu at (143.5, 84.0)
- added C12: 1u, Capacitor_SMD:C_0402_1005Metric, F.Cu at (142.5, 86.2)
- added C13: 1u, Capacitor_SMD:C_0402_1005Metric, F.Cu at (143.5, 83.0)
- added C14: 100n, Capacitor_SMD:C_0402_1005Metric, F.Cu at (144.2, 86.2)
- added C15: 1u, Capacitor_SMD:C_0402_1005Metric, F.Cu at (139.2, 83.8)
- added C16: 7p, Capacitor_SMD:C_0402_1005Metric, F.Cu at (151.5, 98.3)
- added C17: 7p, Capacitor_SMD:C_0402_1005Metric, F.Cu at (151.5, 100.2)
- added C18: 100n, Capacitor_SMD:C_0402_1005Metric, F.Cu at (150.8, 92.8)
- added C19: 10p, Capacitor_SMD:C_0402_1005Metric, F.Cu at (136.6, 69.9)
- added C2: 100n, Capacitor_SMD:C_0402_1005Metric, F.Cu at (150.5, 100.5)
- added C20: 20p, Capacitor_SMD:C_0402_1005Metric, F.Cu at (151.0, 95.5)
- added C21: 20p, Capacitor_SMD:C_0402_1005Metric, F.Cu at (151.0, 94.2)
- added C22: 100n, Capacitor_SMD:C_0402_1005Metric, F.Cu at (143.5, 81.5)
- added C23: 100n, Capacitor_SMD:C_0402_1005Metric, F.Cu at (145.4, 76.3)
- added C24: 100n, Capacitor_SMD:C_0402_1005Metric, F.Cu at (148.4, 68.6)
- added C25: 10p, Capacitor_SMD:C_0402_1005Metric, F.Cu at (134.6, 69.9)
- added C26: 10n, Capacitor_SMD:C_0402_1005Metric, F.Cu at (145.5, 67.0)
- added C27: 10p, Capacitor_SMD:C_0402_1005Metric, F.Cu at (151.9, 69.9)
- added C28: 10p, Capacitor_SMD:C_0402_1005Metric, F.Cu at (149.9, 69.9)
- added C29: 100n, Capacitor_SMD:C_0402_1005Metric, F.Cu at (159.0, 81.3)
- added C3: 100n, Capacitor_SMD:C_0402_1005Metric, F.Cu at (150.5, 97.8)
- added C30: 100n, Capacitor_SMD:C_0402_1005Metric, F.Cu at (164.0, 68.8)
- added C31: 100n, Capacitor_SMD:C_0402_1005Metric, F.Cu at (161.0, 76.2)
- added C32: 10n, Capacitor_SMD:C_0402_1005Metric, F.Cu at (161.0, 67.0)
- added C33: 10p, Capacitor_SMD:C_0402_1005Metric, F.Cu at (121.0, 69.6)
- added C34: 10p, Capacitor_SMD:C_0402_1005Metric, F.Cu at (119.0, 69.6)
- added C35: 100n, Capacitor_SMD:C_0402_1005Metric, F.Cu at (128.0, 81.5)
- added C36: 100n, Capacitor_SMD:C_0402_1005Metric, F.Cu at (133.0, 68.4)
- added C37: 100n, Capacitor_SMD:C_0402_1005Metric, F.Cu at (130.0, 76.1)
- added C38: 10n, Capacitor_SMD:C_0402_1005Metric, F.Cu at (130.0, 67.0)
- added C39: 100n, Capacitor_SMD:C_0402_1005Metric, F.Cu at (129.2, 111.0)
- added C4: 100n, Capacitor_SMD:C_0402_1005Metric, F.Cu at (141.0, 86.2)
- added C40: 10n, Capacitor_SMD:C_0402_1005Metric, F.Cu at (119.8, 111.0)
- added C41: 100n, Capacitor_SMD:C_0402_1005Metric, F.Cu at (121.8, 108.0)
- added C42: 100n, Capacitor_SMD:C_0402_1005Metric, F.Cu at (121.8, 84.6)
- added C43: 100n, Capacitor_SMD:C_0402_1005Metric, F.Cu at (129.2, 87.6)
- added C44: 10n, Capacitor_SMD:C_0402_1005Metric, F.Cu at (119.8, 87.6)
- added C45: 100n, Capacitor_SMD:C_0402_1005Metric, F.Cu at (121.7, 96.1)
- added C46: 100n, Capacitor_SMD:C_0402_1005Metric, F.Cu at (129.2, 99.1)
- added C47: 10n, Capacitor_SMD:C_0402_1005Metric, F.Cu at (119.8, 99.1)
- added C5: 100n, Capacitor_SMD:C_0402_1005Metric, F.Cu at (135.0, 86.8)
- added C6: 100n, Capacitor_SMD:C_0402_1005Metric, F.Cu at (131.8, 95.0)
- added C7: 100n, Capacitor_SMD:C_0402_1005Metric, F.Cu at (131.8, 101.5)
- added C8: 100n, Capacitor_SMD:C_0402_1005Metric, F.Cu at (140.9, 105.5)
- added C9: 100n, Capacitor_SMD:C_0402_1005Metric, F.Cu at (147.0, 105.2)
- added D1: LED, LED_SMD:LED_0402_1005Metric, F.Cu at (160.5, 102.5)
- added D2: LED, LED_SMD:LED_0402_1005Metric, F.Cu at (146.5, 107.5)
- added FB1: 120R, Inductor_SMD:L_0603_1608Metric, F.Cu at (141.8, 83.2)
- added FID1: Fiducial, Fiducial:Fiducial_0.5mm_Mask1.5mm, F.Cu at (167.2, 116.2)
- added FID2: Fiducial, Fiducial:Fiducial_0.5mm_Mask1.5mm, F.Cu at (115.0, 64.0)
- added FID3: Fiducial, Fiducial:Fiducial_0.5mm_Mask1.5mm, F.Cu at (120.0, 116.0)
- added J1: TagConnect_TC2030, Connector:Tag-Connect_TC2030-IDC-FP_2x03_P1.27mm_Vertical, F.Cu at (134.9, 109.7)
- added J10: Conn_01x04_Pin, Connector_PinHeader_2.54mm:PinHeader_1x04_P2.54mm_Vertical, F.Cu at (141.9, 64.0)
- added J11: Conn_01x04_Pin, Connector_PinHeader_2.54mm:PinHeader_1x04_P2.54mm_Vertical, F.Cu at (126.2, 64.1)
- added J12: Conn_01x02_Pin, Connector_PinHeader_2.54mm:PinHeader_1x02_P2.54mm_Vertical, F.Cu at (116.2, 80.0)
- added J2: Conn_01x04_Pin, Connector_PinHeader_2.54mm:PinHeader_1x04_P2.54mm_Vertical, F.Cu at (161.0, 92.8)
- added J3: Conn_01x04_Pin, Connector_PinHeader_2.54mm:PinHeader_1x04_P2.54mm_Vertical, F.Cu at (160.1, 111.0)
- added J4: Conn_01x06_Pin, Connector_PinHeader_2.54mm:PinHeader_1x06_P2.54mm_Horizontal, F.Cu at (165.0, 82.7)
- added J5: Conn_01x06_Pin, Connector_PinHeader_2.54mm:PinHeader_1x06_P2.54mm_Horizontal, F.Cu at (165.0, 99.7)
- added J6: Conn_01x04_Pin, Connector_PinHeader_2.54mm:PinHeader_1x04_P2.54mm_Vertical, F.Cu at (116.3, 114.8)
- added J7: Conn_01x04_Pin, Connector_PinHeader_2.54mm:PinHeader_1x04_P2.54mm_Vertical, F.Cu at (116.2, 91.5)
- added J8: Conn_01x04_Pin, Connector_PinHeader_2.54mm:PinHeader_1x04_P2.54mm_Vertical, F.Cu at (116.2, 102.9)
- added J9: Conn_01x04_Pin, Connector_PinHeader_2.54mm:PinHeader_1x04_P2.54mm_Vertical, F.Cu at (157.2, 64.0)
- added R1: 390R, Resistor_SMD:R_0402_1005Metric, F.Cu at (155.2, 92.0)
- added R10: 60R, Resistor_SMD:R_0402_1005Metric, F.Cu at (128.5, 67.5)
- added R11: 60R, Resistor_SMD:R_0402_1005Metric, F.Cu at (119.8, 110.0)
- added R12: 60R, Resistor_SMD:R_0402_1005Metric, F.Cu at (119.8, 112.0)
- added R13: 60R, Resistor_SMD:R_0402_1005Metric, F.Cu at (119.8, 86.6)
- added R14: 60R, Resistor_SMD:R_0402_1005Metric, F.Cu at (119.8, 88.6)
- added R15: 60R, Resistor_SMD:R_0402_1005Metric, F.Cu at (119.8, 98.1)
- added R16: 60R, Resistor_SMD:R_0402_1005Metric, F.Cu at (119.8, 100.1)
- added R17: 1K, Resistor_SMD:R_0402_1005Metric, F.Cu at (155.0, 107.8)
- added R18: 1K, Resistor_SMD:R_0402_1005Metric, F.Cu at (157.5, 107.8)
- added R19: 10K, Resistor_SMD:R_0402_1005Metric, F.Cu at (139.0, 73.5)
- added R2: 10K, Resistor_SMD:R_0402_1005Metric, F.Cu at (145.2, 105.8)
- added R20: 10K, Resistor_SMD:R_0402_1005Metric, F.Cu at (154.5, 73.8)
- added R21: 10K, Resistor_SMD:R_0402_1005Metric, F.Cu at (123.5, 73.5)
- added R3: 1K, Resistor_SMD:R_0402_1005Metric, F.Cu at (158.5, 102.5)
- added R4: 1K, Resistor_SMD:R_0402_1005Metric, F.Cu at (148.5, 106.0)
- added R5: 60R, Resistor_SMD:R_0402_1005Metric, F.Cu at (147.0, 67.5)
- added R6: 60R, Resistor_SMD:R_0402_1005Metric, F.Cu at (144.0, 67.5)
- added R7: 60R, Resistor_SMD:R_0402_1005Metric, F.Cu at (162.5, 67.5)
- added R8: 60R, Resistor_SMD:R_0402_1005Metric, F.Cu at (159.5, 67.5)
- added R9: 60R, Resistor_SMD:R_0402_1005Metric, F.Cu at (131.5, 67.5)
- added SW2: SW_SPDT_321, Button_Switch_SMD:SW_SPDT_PCM12, F.Cu at (144.5, 110.5)
- added SW3: SW_Push, Button_Switch_SMD:SW_SPST_CK_RS282G05A3, F.Cu at (153.5, 85.2)
- added U1: STM32G474QETx, Package_QFP:LQFP-128_14x14mm_P0.4mm, F.Cu at (141.0, 96.0)
- added U10: TJA1051T-3, Package_SO:SOIC-8_3.9x4.9mm_P1.27mm, F.Cu at (125.0, 99.1)
- added U2: MCP2517FD-xSL, Package_SO:SOIC-14_3.9x8.7mm_P1.27mm, F.Cu at (154.0, 78.0)
- added U3: MCP2517FD-xSL, Package_SO:SOIC-14_3.9x8.7mm_P1.27mm, F.Cu at (138.5, 78.0)
- added U4: TJA1051T-3, Package_SO:SOIC-8_3.9x4.9mm_P1.27mm, F.Cu at (145.4, 72.0)
- added U5: TJA1051T-3, Package_SO:SOIC-8_3.9x4.9mm_P1.27mm, F.Cu at (161.0, 72.0)
- added U6: MCP2517FD-xSL, Package_SO:SOIC-14_3.9x8.7mm_P1.27mm, F.Cu at (123.0, 78.0)
- added U7: TJA1051T-3, Package_SO:SOIC-8_3.9x4.9mm_P1.27mm, F.Cu at (130.0, 71.9)
- added U8: TJA1051T-3, Package_SO:SOIC-8_3.9x4.9mm_P1.27mm, F.Cu at (125.0, 111.0)
- added U9: TJA1051T-3, Package_SO:SOIC-8_3.9x4.9mm_P1.27mm, F.Cu at (125.0, 87.6)
- added Y1: 32.768KHz, Crystal:Crystal_SMD_3215-2Pin_3.2x1.5mm, F.Cu at (153.2, 99.2)
- added Y2: 24MHz, Crystal:Crystal_SMD_TXC_7M-4Pin_3.2x2.5mm, F.Cu at (154.5, 94.8)
- added Y3: 40MHz, Crystal:Crystal_SMD_TXC_7M-4Pin_3.2x2.5mm, F.Cu at (135.6, 72.4)
- added Y4: 40MHz, Crystal:Crystal_SMD_TXC_7M-4Pin_3.2x2.5mm, F.Cu at (150.9, 72.4)
- added Y5: 40MHz, Crystal:Crystal_SMD_TXC_7M-4Pin_3.2x2.5mm, F.Cu at (120.0, 72.1)
Routing:
- net +5V: track 0.00 -> 183.0 mm, vias 0 -> 7
- net GND: track 0.00 -> 175.1 mm, vias 0 -> 89
- net +3.3V: track 0.00 -> 139.7 mm, vias 0 -> 58
- net /SWD_NRST: track 0.00 -> 66.5 mm, vias 0 -> 4
- net SPI1_MISO: track 0.00 -> 40.0 mm, vias 0 -> 3
- net SPI1_SCK: track 0.00 -> 39.2 mm, vias 0 -> 3
- net EXTI3: track 0.00 -> 38.7 mm
- net EXTI1: track 0.00 -> 37.8 mm, vias 0 -> 2
- net /SPI2_MOSI: track 0.00 -> 37.5 mm, vias 0 -> 1
- net /SPI2_MISO: track 0.00 -> 37.4 mm, vias 0 -> 1
- net SPI3_SCK: track 0.00 -> 33.7 mm, vias 0 -> 2
- net SPI3_MOSI: track 0.00 -> 33.6 mm, vias 0 -> 2
- net SPI3_MISO: track 0.00 -> 31.9 mm, vias 0 -> 2
- net SPI3_CS1: track 0.00 -> 31.2 mm, vias 0 -> 2
- net EXTI2: track 0.00 -> 27.6 mm
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- added copper zone on In2.Cu, net +3.3V
- added copper zone on In1.Cu, net GND
Other:
- board outline added: 56.2 x 57 mm
- board text added: "BOOT0 SW"
- board text added: "CAN1"
- board text added: "CAN2"
- board text added: "CAN3"
- board text added: "CAN4"
- board text added: "CAN5"
- board text added: "CAN6"
- board text added: "I2C"
- board text added: "JMSN2519"
- board text added: "MRLMbdv1.0"
- board text added: "PWR"
- board text added: "Raspberry Pi SPI Channels"
- board text added: "SWD"
- board text added: "UART"

Commit message: PCB Update
Parts:
- removed C12: 1u, Capacitor_SMD:C_0402_1005Metric
- removed C30: 100n, Capacitor_SMD:C_0402_1005Metric
- added 3.3V: Conn_01x02_Pin, Connector_PinHeader_2.54mm:PinHeader_1x02_P2.54mm_Vertical, F.Cu at (166.0, 76.8)
- added D3: LED, LED_SMD:LED_0402_1005Metric, F.Cu at (115.2, 72.0)
- added R22: 10K, Resistor_SMD:R_0402_1005Metric, F.Cu at (115.2, 70.0)
- moved D1 2.02 mm to (158.8, 101.5)
- moved R3 2.02 mm to (156.8, 101.5)
- moved FID1 0.50 mm to (167.8, 116.2)
- renumbered J12 to 5V
Routing:
- net +3.3V: track 139.7 -> 127.2 mm, vias 58 -> 63
- net +5V: track 183.0 -> 191.3 mm
- net Net-(D3-A): track 0.00 -> 1.02 mm
- net GND: track 175.1 -> 175.8 mm, vias 89 -> 93
- added copper zone on F.Cu, net +3.3V
- added copper zone on F.Cu, net GND
Other:
- board size 56.2 x 57 mm -> 56.8 x 57 mm
- board text added: "3.3V"
- board text added: "5V"
- board text added: "CAN+"
- board text added: "CAN-"
- board text added: "CS"
- board text added: "GND"
- board text added: "MISO"
- board text added: "MOSI"
- board text added: "PWR 5V"
- board text added: "RST"
- board text added: "RX"
- board text added: "SCK"
- board text added: "SCL"
- board text added: "SDA"
- board text added: "SPI2"
- board text added: "SPI4"
- board text added: "TX"
