File: stm32g474/stm32g474.kicad_sch (KiCad schematic)
At the start: 45 parts, among them J1 TagConnect_TC2030, J10 Conn_01x04_Pin, J11 Conn_01x04_Pin, J2 Conn_01x04_Pin, J3 Conn_01x04_Pin, J4 Conn_01x06_Pin, J5 Conn_01x06_Pin, J6 Conn_01x04_Pin, J7 Conn_01x04_Pin, J8 Conn_01x04_Pin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

Commit message: pcb update
Parts:
- added FID1, FID2, FID3: Fiducial, Fiducial:Fiducial_0.5mm_Mask1.5mm, symbol Mechanical:Fiducial
- added J12: Conn_01x02_Pin, Connector_PinHeader_2.54mm:PinHeader_1x02_P2.54mm_Vertical, symbol Connector:Conn_01x02_Pin
Connections:
- net SWO is gone; now on net SWD_SWO: U1.118 (PB3)
- net EXTI1: now also U1.25 (PC3); no longer U1.23 (PC1)
- net EXTI3: now also U1.23 (PC1); no longer U1.25 (PC3)
- net GND: now also J12.2 (Pin_2)
- net HSE_OUT: now also C21.1, R1.1, Y2.2
- new net +5V: J12.1 (Pin_1)

Commit message: PCB Update
Parts:
- added D3: LED, LED_SMD:LED_0402_1005Metric, symbol Device:LED
- added J13: Conn_01x02_Pin, Connector_PinHeader_2.54mm:PinHeader_1x02_P2.54mm_Vertical, symbol Connector:Conn_01x02_Pin
- added R22: 10K, Resistor_SMD:R_0402_1005Metric, symbol Device:R
Connections:
- net +3.3V: now also J13.1 (Pin_1)
- net +5V: now also D3.2 (A)
- net GND: now also J13.2 (Pin_2), R22.1
- new net: D3.1 (K), R22.2
Other:
- note added: "5V power check"

Commit message: PCB Update
Other:
- note added: "Power input"
- note removed: "Need to choose specific crystals (everywhere) -caps will change"
- moved on the sheet: FID1, FID2, FID3, J13
Changed lines of the file:
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@@
 	)
 	(rectangle
+		(start 81.28 175.26)
+		(end 127 187.96)
+		(stroke
+			(width 0)
+			(type default)
+		)
+		(fill
+			(type none)
+		)
+	)
+	(rectangle
 		(start 80.01 41.91)
 		(end 111.76 67.31)
@@
 		)
 	)
+	(text "Power input"
+		(exclude_from_sim no)
+		(at 103.632 189.992 0)
+		(effects
+			(font
+				(size 1.27 1.27)
+			)
+		)
+	)
 	(text "CAN3"
 		(exclude_from_sim no)
@@
 		)
 	)
-	(text "Need to choose specific crystals (everywhere) -caps will change"
-		(exclude_from_sim no)
-		(at 101.6 168.656 0)
-		(effects
-			(font
-				(size 1.27 1.27)
-				(thickness 0.254)
-				(bold yes)
-			)
-		)
-	)
 	(junction
 		(at 106.68 148.59)
@@
 	(symbol
 		(lib_id "power:GND")
-		(at 269.24 154.94 90)
+		(at 96.52 185.42 90)
 		(unit 1)
 		(exclude_from_sim no)
@@
 		(fields_autoplaced yes)
 		(property "Reference" "#PWR098"
-			(at 275.59 154.94 0)
+			(at 102.87 185.42 0)
 			(effects
 				(font
@@
 		)
 		(property "Value" "GND"
-			(at 273.05 154.9399 90)
+			(at 100.33 185.4199 90)
 			(effects
 				(font
@@
 		)
 		(property "Footprint" ""
-			(at 269.24 154.94 0)
+			(at 96.52 185.42 0)
 			(effects
 				(font
@@
 		)
 		(property "Datasheet" ""
-			(at 269.24 154.94 0)
+			(at 96.52 185.42 0)
 			(effects
 				(font
@@
 		)
 		(property "Description" "Power symbol creates a global label with name \"GND\" , ground"
-			(at 269.24 154.94 0)
+			(at 96.52 185.42 0)
 			(effects
 				(font
@@
 	(symbol
 		(lib_id "power:+3.3V")
-		(at 269.24 152.4 270)
+		(at 96.52 182.88 270)
 		(unit 1)
 		(exclude_from_sim no)
@@
 		(fields_autoplaced yes)
 		(property "Reference" "#PWR097"
-			(at 265.43 152.4 0)
+			(at 92.71 182.88 0)
 			(effects
 				(font
@@
 		)
 		(property "Value" "+3.3V"
-			(at 273.05 152.3999 90)
+			(at 100.33 182.8799 90)
 			(effects
 				(font
@@
 		)
 		(property "Footprint" ""
-			(at 269.24 152.4 0)
+			(at 96.52 182.88 0)
 			(effects
 				(font
@@
 		)
 		(property "Datasheet" ""
-			(at 269.24 152.4 0)
+			(at 96.52 182.88 0)
 			(effects
 				(font
@@
 		)
 		(property "Description" "Power symbol creates a global label with name \"+3.3V\""
-			(at 269.24 152.4 0)
+			(at 96.52 182.88 0)
 			(effects
 				(font
@@
 	(symbol
 		(lib_id "Connector:Conn_01x02_Pin")
-		(at 264.16 152.4 0)
+		(at 91.44 182.88 0)
 		(unit 1)
 		(exclude_from_sim no)
@@
 		(fields_autoplaced yes)
 		(property "Reference" "J13"
-			(at 264.795 147.32 0)
+			(at 92.075 177.8 0)
 			(effects
 				(font
@@
 		)
 		(property "Value" "Conn_01x02_Pin"
-			(at 264.795 149.86 0)
+			(at 92.075 180.34 0)
 			(effects
 				(font
@@
 		)
 		(property "Footprint" "Connector_PinHeader_2.54mm:PinHeader_1x02_P2.54mm_Vertical"
-			(at 264.16 152.4 0)
+			(at 91.44 182.88 0)
 			(effects
 				(font
@@
 		)
 		(property "Datasheet" "~"
-			(at 264.16 152.4 0)
+			(at 91.44 182.88 0)
 			(effects
 				(font
@@
 		)
 		(property "Description" "Generic connector, single row, 01x02, script generated"
-			(at 264.16 152.4 0)
+			(at 91.44 182.88 0)
 			(effects
 				(font
@@
 	(symbol
 		(lib_id "Mechanical:Fiducial")
-		(at 68.58 190.5 0)
+		(at 68.58 161.29 0)
 		(unit 1)
 		(exclude_from_sim no)
@@
 		(fields_autoplaced yes)
 		(property "Reference" "FID3"
-			(at 71.12 189.2299 0)
+			(at 71.12 160.0199 0)
 			(effects
 				(font
@@
 		)
 		(property "Value" "Fiducial"
-			(at 71.12 191.7699 0)
+			(at 71.12 162.5599 0)
 			(effects
 				(font
@@
 		)
 		(property "Footprint" "Fiducial:Fiducial_0.5mm_Mask1.5mm"
-			(at 68.58 190.5 0)
+			(at 68.58 161.29 0)
 			(effects
 				(font
@@
 		)
 		(property "Datasheet" "~"
-			(at 68.58 190.5 0)
+			(at 68.58 161.29 0)
 			(effects
 				(font
@@
 		)
 		(property "Description" "Fiducial Marker"
-			(at 68.58 190.5 0)
+			(at 68.58 161.29 0)
 			(effects
 				(font
@@
 	(symbol
 		(lib_id "Mechanical:Fiducial")
-		(at 68.58 184.15 0)
+		(at 68.58 154.94 0)
 		(unit 1)
 		(exclude_from_sim no)
@@
 		(fields_autoplaced yes)
 		(property "Reference" "FID2"
-			(at 71.12 182.8799 0)
+			(at 71.12 153.6699 0)
 			(effects
 				(font
@@
 		)
 		(property "Value" "Fiducial"
-			(at 71.12 185.4199 0)
+			(at 71.12 156.2099 0)
 			(effects
 				(font
@@
 		)
 		(property "Footprint" "Fiducial:Fiducial_0.5mm_Mask1.5mm"
-			(at 68.58 184.15 0)
+			(at 68.58 154.94 0)
 			(effects
 				(font
@@
 		)
 		(property "Datasheet" "~"
-			(at 68.58 184.15 0)
+			(at 68.58 154.94 0)
 			(effects
 				(font
@@
 		)
 		(property "Description" "Fiducial Marker"
-			(at 68.58 184.15 0)
+			(at 68.58 154.94 0)
 			(effects
 				(font
@@
 	(symbol
 		(lib_id "Mechanical:Fiducial")
-		(at 68.58 177.8 0)
+		(at 68.58 148.59 0)
 		(unit 1)
 		(exclude_from_sim no)
@@
 		(fields_autoplaced yes)
 		(property "Reference" "FID1"
-			(at 71.12 176.5299 0)
+			(at 71.12 147.3199 0)
 			(effects
 				(font
@@
 		)
 		(property "Value" "Fiducial"
-			(at 71.12 179.0699 0)
+			(at 71.12 149.8599 0)
 			(effects
 				(font
@@
 		)
 		(property "Footprint" "Fiducial:Fiducial_0.5mm_Mask1.5mm"
-			(at 68.58 177.8 0)
+			(at 68.58 148.59 0)
 			(effects
 				(font
@@
 		)
 		(property "Datasheet" "~"
-			(at 68.58 177.8 0)
+			(at 68.58 148.59 0)
 			(effects
 				(font
@@
 		)
 		(property "Description" "Fiducial Marker"
-			(at 68.58 177.8 0)
+			(at 68.58 148.59 0)
 			(effects
 				(font
